File: ssc.sch (KiCad schematic (older format))
At the start: 26 parts, among them J1 IRQ ENABLE, J2 RS-232 OUT, P1 A2Bus, U1 74HC245, U2 28C256, U3 1.8432M, U4 SSCGLU, U5 W65C51NxP, U6 MAX3232, U7 MAX3232

Commit message: - Updated schematic, mostly tweaks to make layout easier. - Updated GAL equations - Add PCBNew layout for initial test run
Parts:
- removed C14, C16, C8: 0.1u, symbol Device:C_Small
- added C14, C16: 1u, Capacitor_THT:CP_Radial_D5.0mm_P2.50mm, symbol Device:CP_Small
- C1, C2, C3, C4, C5, C6, C7: footprint (none) -> Capacitor_THT:C_Disc_D4.3mm_W1.9mm_P5.00mm
- C10, C11, C12, C13, C15, C9: value 0.1u -> 1u; footprint (none) -> Capacitor_THT:CP_Radial_D5.0mm_P2.50mm; symbol Device:C_Small -> Device:CP_Small
- J1: footprint (none) -> Connector_PinHeader_2.54mm:PinHeader_1x02_P2.54mm_Vertical
- J2: footprint (none) -> Connector_PinHeader_2.54mm:PinHeader_2x05_P2.54mm_Vertical; symbol Connector_Generic:Conn_02x05_Odd_Even -> ssc:Conn_PC_MB_Serial
- P1: footprint (none) -> Apple2-Bus:Male_Card-Edge_50_pin__100_mil
- U1: value 74HC245 -> 74HCT245; footprint (none) -> Package_DIP:DIP-20_W7.62mm_Socket
- U2, U5: footprint (none) -> Package_DIP:DIP-28_W15.24mm_Socket
- U3: footprint (none) -> Package_DIP:DIP-8_W7.62mm_Socket
- U4: footprint Package_DIP:DIP-24_W7.62mm -> Package_DIP:DIP-24_W7.62mm_Socket
- U6, U7: footprint (none) -> Package_DIP:DIP-16_W7.62mm_Socket
Connections:
- net D0: now also U1.9 (A7); no longer U1.2 (A0)
- net D1: now also U1.8 (A6); no longer U1.3 (A1)
- net D2: now also U1.7 (A5); no longer U1.4 (A2)
- net D3: now also U1.6 (A4); no longer U1.5 (A3)
- net D4: now also U1.5 (A3); no longer U1.6 (A4)
- net D5: now also U1.4 (A2); no longer U1.7 (A5)
- net D6: now also U1.3 (A1); no longer U1.8 (A6)
- net D7: now also U1.2 (A0); no longer U1.9 (A7)
- net GND: now also C13.1, C14.1, C16.2; no longer C13.2
- net MD0: now reaches U1.11 (B7)
- net MD0: now also P1.49 (D0); no longer P1.42 (D7)
- net MD1: now reaches U1.12 (B6)
- net MD1: now also P1.48 (D1); no longer P1.43 (D6)
- net MD2: now reaches U1.13 (B5)
- net MD2: now also P1.47 (D2); no longer P1.44 (D5)
- net MD3: now reaches U1.14 (B4)
- net MD3: now also P1.46 (D3); no longer P1.45 (D4)
- net MD4: now reaches U1.15 (B3)
- net MD4: now also P1.45 (D4); no longer P1.46 (D3)
- net MD5: now reaches U1.16 (B2)
- net MD5: now also P1.44 (D5); no longer P1.47 (D2)
- net MD6: now reaches U1.17 (B1)
- net MD6: now also P1.43 (D6); no longer P1.48 (D1)
- net MD7: now reaches U1.18 (B0)
- net MD7: now also P1.42 (D7); no longer P1.49 (D0)
- net at U6.6 (VS-): now also C13.2; no longer C13.1
- net at U7.2 (VS+): now also C16.1
- net at U7.6 (VS-): now also C14.2
- net CTS: no longer names the net of U4.2 (CTS), U5.9 (~CTS), U6.9 (R2OUT)
- net CTS: no longer J2.8 (Pin_8), U6.8 (R2IN)
- net DCD: no longer names the net of J2.1 (DCD), U7.8 (R2IN)
- net DSR: no longer names the net of J2.6 (DSR), U7.13 (R1IN)
- net DTR: no longer names the net of J2.4 (DTR), U7.14 (T1OUT)
- net RTS: no longer names the net of J2.7 (RTS), U6.7 (T2OUT)
- net RxD: no longer names the net of J2.2 (RxD), U6.13 (R1IN)
- net TxD: no longer names the net of J2.3 (TxD), U6.14 (T1OUT)
- new net: J2.8 (CTS), U6.8 (R2IN)
- no-connect marks 23 -> 22
Other:
- moved on the sheet: C1, C2, C3, C4, C5, C6, C7, P1, U1, U2, U3
